File: Mini-Traveller-Keyboard.sch (KiCad schematic (older format))
At the start: 114 parts, among them P1 USB_C_Receptacle_USB2.0, SW1 SW_Push, U1 ATmega32U4-AU, Y1 16MHz

Commit message: Finished main PCB design, waiting on silk
Parts:
- P1: symbol Connector:USB_C_Receptacle_USB2.0 -> Mini-Traveller-Keyboard-rescue:USB_C_Receptacle_USB2.0-Connector
Changed lines of the file:
@@
 D-
 $Comp
-L Connector:USB_C_Receptacle_USB2.0 P1
+L Mini-Traveller-Keyboard-rescue:USB_C_Receptacle_USB2.0-Connector P1
 U 1 1 5F7D3E13
 P -850 1800
@@
 Text GLabel 4850 3750 0    50   Input ~ 0
 Row3
+Text GLabel 3400 2800 2    50   Input ~ 0
+Col0
+Text GLabel 3400 3000 2    50   Input ~ 0
+Col1
+Text GLabel 3400 3100 2    50   Input ~ 0
+Col2
+Text GLabel 3400 1600 2    50   Input ~ 0
+Col3
+Text GLabel 3400 1700 2    50   Input ~ 0
+Col4
+Text GLabel 3400 1800 2    50   Input ~ 0
+Col5
+Text GLabel 3400 3700 2    50   Input ~ 0
+Col7
+Text GLabel 3400 3800 2    50   Input ~ 0
+Col8
+Text GLabel 3400 3900 2    50   Input ~ 0
+Col9
+Text GLabel 3400 1500 2    50   Input ~ 0
+Col11
+Text GLabel 3400 4100 2    50   Input ~ 0
+Col10
+Text GLabel 3400 3600 2    50   Input ~ 0
+Col6
 $EndSCHEMATC

Commit message: files
Parts:
- added D49, D50, D51: WS2812B, LED_SMD:LED_WS2812B_PLCC4_5.0x5.0mm_P3.2mm, symbol LED:WS2812B
- MX1, MX10, MX11, MX12, MX13, MX14, MX15, MX16, MX17, MX18, MX19, MX2, MX20, MX21, MX22, MX23, MX24, MX25, MX26, MX27, MX28, MX29, MX3, MX30, MX31, MX32, MX33, MX34, MX35, MX36, MX37, MX38, MX39, MX4, MX40, MX41, MX42, MX43, MX44, MX45, MX46, MX47, MX48, MX5, MX6, MX7, MX8, MX9: symbol MX_Alps_Hybrid:MX-NoLED -> Mini-Traveller-Keyboard-rescue:MX-NoLED-MX_Alps_Hybrid
Connections:
- net +5V: now also D51.1 (VDD)
- net GND: now also D49.3 (VSS), D50.3 (VSS), D51.3 (VSS)
- new net: D50.2 (DOUT), D51.4 (DIN)
- new net: D49.2 (DOUT), D50.4 (DIN)
Changed lines of the file:
@@
 	-250 2200 1700 2200
 $Comp
-L MX_Alps_Hybrid:MX-NoLED MX1
+L Mini-Traveller-Keyboard-rescue:MX-NoLED-MX_Alps_Hybrid MX1
 U 1 1 5F822F44
 P 5300 1450
@@
 	5100 1600 5250 1600
 $Comp
-L MX_Alps_Hybrid:MX-NoLED MX5
+L Mini-Traveller-Keyboard-rescue:MX-NoLED-MX_Alps_Hybrid MX5
 U 1 1 5F828EE1
 P 5800 1450
@@
 	5600 1600 5750 1600
 $Comp
-L MX_Alps_Hybrid:MX-NoLED MX9
+L Mini-Traveller-Keyboard-rescue:MX-NoLED-MX_Alps_Hybrid MX9
 U 1 1 5F82F6DD
 P 6300 1450
@@
 	6100 1600 6250 1600
 $Comp
-L MX_Alps_Hybrid:MX-NoLED MX13
+L Mini-Traveller-Keyboard-rescue:MX-NoLED-MX_Alps_Hybrid MX13
 U 1 1 5F82F6EA
 P 6800 1450
@@
 	6600 1600 6750 1600
 $Comp
-L MX_Alps_Hybrid:MX-NoLED MX17
+L Mini-Traveller-Keyboard-rescue:MX-NoLED-MX_Alps_Hybrid MX17
 U 1 1 5F83395C
 P 7300 1450
@@
 	7100 1600 7250 1600
 $Comp
-L MX_Alps_Hybrid:MX-NoLED MX21
+L Mini-Traveller-Keyboard-rescue:MX-NoLED-MX_Alps_Hybrid MX21
 U 1 1 5F833969
 P 7800 1450
@@
 	7600 1600 7750 1600
 $Comp
-L MX_Alps_Hybrid:MX-NoLED MX25
+L Mini-Traveller-Keyboard-rescue:MX-NoLED-MX_Alps_Hybrid MX25
 U 1 1 5F833976
 P 8300 1450
@@
 	8100 1600 8250 1600
 $Comp
-L MX_Alps_Hybrid:MX-NoLED MX29
+L Mini-Traveller-Keyboard-rescue:MX-NoLED-MX_Alps_Hybrid MX29
 U 1 1 5F833983
 P 8800 1450
@@
 	8600 1600 8750 1600
 $Comp
-L MX_Alps_Hybrid:MX-NoLED MX33
+L Mini-Traveller-Keyboard-rescue:MX-NoLED-MX_Alps_Hybrid MX33
 U 1 1 5F83810B
 P 9300 1450
@@
 	9100 1600 9250 1600
 $Comp
-L MX_Alps_Hybrid:MX-NoLED MX37
+L Mini-Traveller-Keyboard-rescue:MX-NoLED-MX_Alps_Hybrid MX37
 U 1 1 5F838118
 P 9800 1450
@@
 	9600 1600 9750 1600
 $Comp
-L MX_Alps_Hybrid:MX-NoLED MX41
+L Mini-Traveller-Keyboard-rescue:MX-NoLED-MX_Alps_Hybrid MX41
 U 1 1 5F838125
 P 10300 1450
@@
 	10100 1600 10250 1600
 $Comp
-L MX_Alps_Hybrid:MX-NoLED MX45
+L Mini-Traveller-Keyboard-rescue:MX-NoLED-MX_Alps_Hybrid MX45
 U 1 1 5F838132
 P 10800 1450
@@
 	10600 1600 10750 1600
 $Comp
-L MX_Alps_Hybrid:MX-NoLED MX2
+L Mini-Traveller-Keyboard-rescue:MX-NoLED-MX_Alps_Hybrid MX2
 U 1 1 5F866319
 P 5300 2100
@@
 	5100 2250 5250 2250
 $Comp
-L MX_Alps_Hybrid:MX-NoLED MX6
+L Mini-Traveller-Keyboard-rescue:MX-NoLED-MX_Alps_Hybrid MX6
 U 1 1 5F866326
 P 5800 2100
@@
 	5600 2250 5750 2250
 $Comp
-L MX_Alps_Hybrid:MX-NoLED MX10
+L Mini-Traveller-Keyboard-rescue:MX-NoLED-MX_Alps_Hybrid MX10
 U 1 1 5F866333
 P 6300 2100
@@
 	6100 2250 6250 2250
 $Comp
-L MX_Alps_Hybrid:MX-NoLED MX14
+L Mini-Traveller-Keyboard-rescue:MX-NoLED-MX_Alps_Hybrid MX14
 U 1 1 5F866340
 P 6800 2100
@@
 	6600 2250 6750 2250
 $Comp
-L MX_Alps_Hybrid:MX-NoLED MX18
+L Mini-Traveller-Keyboard-rescue:MX-NoLED-MX_Alps_Hybrid MX18
 U 1 1 5F86634D
 P 7300 2100
@@
 	7100 2250 7250 2250
 $Comp
-L MX_Alps_Hybrid:MX-NoLED MX22
+L Mini-Traveller-Keyboard-rescue:MX-NoLED-MX_Alps_Hybrid MX22
 U 1 1 5F86635A
 P 7800 2100
@@
 	7600 2250 7750 2250
 $Comp
-L MX_Alps_Hybrid:MX-NoLED MX26
+L Mini-Traveller-Keyboard-rescue:MX-NoLED-MX_Alps_Hybrid MX26
 U 1 1 5F866367
 P 8300 2100
@@
 	8100 2250 8250 2250
 $Comp
-L MX_Alps_Hybrid:MX-NoLED MX30
+L Mini-Traveller-Keyboard-rescue:MX-NoLED-MX_Alps_Hybrid MX30
 U 1 1 5F866374
 P 8800 2100
@@
 	8600 2250 8750 2250
 $Comp
-L MX_Alps_Hybrid:MX-NoLED MX34
+L Mini-Traveller-Keyboard-rescue:MX-NoLED-MX_Alps_Hybrid MX34
 U 1 1 5F866381
 P 9300 2100
@@
 	9100 2250 9250 2250
 $Comp
-L MX_Alps_Hybrid:MX-NoLED MX38
+L Mini-Traveller-Keyboard-rescue:MX-NoLED-MX_Alps_Hybrid MX38
 U 1 1 5F86638E
 P 9800 2100
@@
 	9600 2250 9750 2250
 $Comp
-L MX_Alps_Hybrid:MX-NoLED MX42
+L Mini-Traveller-Keyboard-rescue:MX-NoLED-MX_Alps_Hybrid MX42
 U 1 1 5F86639B
 P 10300 2100
@@
 	10100 2250 10250 2250
 $Comp
-L MX_Alps_Hybrid:MX-NoLED MX46
+L Mini-Traveller-Keyboard-rescue:MX-NoLED-MX_Alps_Hybrid MX46
 U 1 1 5F8663A8
 P 10800 2100
@@
 	10600 2250 10750 2250
 $Comp
-L MX_Alps_Hybrid:MX-NoLED MX3
+L Mini-Traveller-Keyboard-rescue:MX-NoLED-MX_Alps_Hybrid MX3
 U 1 1 5F8805BC
 P 5300 2750
@@
 	5100 2900 5250 2900
 $Comp
-L MX_Alps_Hybrid:MX-NoLED MX7
+L Mini-Traveller-Keyboard-rescue:MX-NoLED-MX_Alps_Hybrid MX7
 U 1 1 5F8805C9
 P 5800 2750
@@
 	5600 2900 5750 2900
 $Comp
-L MX_Alps_Hybrid:MX-NoLED MX11
+L Mini-Traveller-Keyboard-rescue:MX-NoLED-MX_Alps_Hybrid MX11
 U 1 1 5F8805D6
 P 6300 2750
@@
 	6100 2900 6250 2900
 $Comp
-L MX_Alps_Hybrid:MX-NoLED MX15
+L Mini-Traveller-Keyboard-rescue:MX-NoLED-MX_Alps_Hybrid MX15
 U 1 1 5F8805E3
 P 6800 2750
@@
 	6600 2900 6750 2900
 $Comp
-L MX_Alps_Hybrid:MX-NoLED MX19
+L Mini-Traveller-Keyboard-rescue:MX-NoLED-MX_Alps_Hybrid MX19
 U 1 1 5F8805F0
 P 7300 2750
@@
 	7100 2900 7250 2900
 $Comp
-L MX_Alps_Hybrid:MX-NoLED MX23
+L Mini-Traveller-Keyboard-rescue:MX-NoLED-MX_Alps_Hybrid MX23
 U 1 1 5F8805FD
 P 7800 2750
@@
 	7600 2900 7750 2900
 $Comp
-L MX_Alps_Hybrid:MX-NoLED MX27
+L Mini-Traveller-Keyboard-rescue:MX-NoLED-MX_Alps_Hybrid MX27
 U 1 1 5F88060A
 P 8300 2750
@@
 	8100 2900 8250 2900
 $Comp
-L MX_Alps_Hybrid:MX-NoLED MX31
+L Mini-Traveller-Keyboard-rescue:MX-NoLED-MX_Alps_Hybrid MX31
 U 1 1 5F880617
 P 8800 2750
@@
 	8600 2900 8750 2900
 $Comp
-L MX_Alps_Hybrid:MX-NoLED MX35
+L Mini-Traveller-Keyboard-rescue:MX-NoLED-MX_Alps_Hybrid MX35
 U 1 1 5F880624
 P 9300 2750
@@
 	9100 2900 9250 2900
 $Comp
-L MX_Alps_Hybrid:MX-NoLED MX39
+L Mini-Traveller-Keyboard-rescue:MX-NoLED-MX_Alps_Hybrid MX39
 U 1 1 5F880631
 P 9800 2750
@@
 	9600 2900 9750 2900
 $Comp
-L MX_Alps_Hybrid:MX-NoLED MX43
+L Mini-Traveller-Keyboard-rescue:MX-NoLED-MX_Alps_Hybrid MX43
 U 1 1 5F88063E
 P 10300 2750
@@
 	10100 2900 10250 2900
 $Comp
-L MX_Alps_Hybrid:MX-NoLED MX47
+L Mini-Traveller-Keyboard-rescue:MX-NoLED-MX_Alps_Hybrid MX47
 U 1 1 5F88064B
 P 10800 2750
@@
 	10600 2900 10750 2900
 $Comp
-L MX_Alps_Hybrid:MX-NoLED MX4
+L Mini-Traveller-Keyboard-rescue:MX-NoLED-MX_Alps_Hybrid MX4
 U 1 1 5F88FC81
 P 5300 3400
@@
 	5100 3550 5250 3550
 $Comp
-L MX_Alps_Hybrid:MX-NoLED MX8
+L Mini-Traveller-Keyboard-rescue:MX-NoLED-MX_Alps_Hybrid MX8
 U 1 1 5F88FC8E
 P 5800 3400
@@
 	5600 3550 5750 3550
 $Comp
-L MX_Alps_Hybrid:MX-NoLED MX12
+L Mini-Traveller-Keyboard-rescue:MX-NoLED-MX_Alps_Hybrid MX12
 U 1 1 5F88FC9B
 P 6300 3400
@@
 	6100 3550 6250 3550
 $Comp
-L MX_Alps_Hybrid:MX-NoLED MX16
+L Mini-Traveller-Keyboard-rescue:MX-NoLED-MX_Alps_Hybrid MX16
 U 1 1 5F88FCA8
 P 6800 3400
@@
 	6600 3550 6750 3550
 $Comp
-L MX_Alps_Hybrid:MX-NoLED MX20
+L Mini-Traveller-Keyboard-rescue:MX-NoLED-MX_Alps_Hybrid MX20
 U 1 1 5F88FCB5
 P 7300 3400
@@
 	7100 3550 7250 3550
 $Comp
-L MX_Alps_Hybrid:MX-NoLED MX24
+L Mini-Traveller-Keyboard-rescue:MX-NoLED-MX_Alps_Hybrid MX24
 U 1 1 5F88FCC2
 P 7800 3400
@@
 	7600 3550 7750 3550
 $Comp
-L MX_Alps_Hybrid:MX-NoLED MX28
+L Mini-Traveller-Keyboard-rescue:MX-NoLED-MX_Alps_Hybrid MX28
 U 1 1 5F88FCCF
 P 8300 3400
@@
 	8100 3550 8250 3550
 $Comp
-L MX_Alps_Hybrid:MX-NoLED MX32
+L Mini-Traveller-Keyboard-rescue:MX-NoLED-MX_Alps_Hybrid MX32
 U 1 1 5F88FCDC
 P 8800 3400
@@
 	8600 3550 8750 3550
 $Comp
-L MX_Alps_Hybrid:MX-NoLED MX36
+L Mini-Traveller-Keyboard-rescue:MX-NoLED-MX_Alps_Hybrid MX36
 U 1 1 5F88FCE9
 P 9300 3400
@@
 	9100 3550 9250 3550
 $Comp
-L MX_Alps_Hybrid:MX-NoLED MX40
+L Mini-Traveller-Keyboard-rescue:MX-NoLED-MX_Alps_Hybrid MX40
 U 1 1 5F88FCF6
 P 9800 3400
@@
 	9600 3550 9750 3550
 $Comp
-L MX_Alps_Hybrid:MX-NoLED MX44
+L Mini-Traveller-Keyboard-rescue:MX-NoLED-MX_Alps_Hybrid MX44
 U 1 1 5F88FD03
 P 10300 3400
@@
 	10100 3550 10250 3550
 $Comp
-L MX_Alps_Hybrid:MX-NoLED MX48
+L Mini-Traveller-Keyboard-rescue:MX-NoLED-MX_Alps_Hybrid MX48
 U 1 1 5F88FD10
 P 10800 3400
@@
 Text GLabel 3400 3600 2    50   Input ~ 0
 Col6
+$Comp
+L LED:WS2812B D51
+U 1 1 5FA23891
+P 7400 4900
+F 0 "D51" H 7744 4946 50  0000 L CNN
+F 1 "WS2812B" H 7744 4855 50  0000 L CNN
+F 2 "LED_SMD:LED_WS2812B_PLCC4_5.0x5.0mm_P3.2mm" H 7450 4600 50  0001 L TNN
+F 3 "https://cdn-shop.adafruit.com/datasheets/WS2812B.pdf" H 7500 4525 50  0001 L TNN
+	1    7400 4900
+	1    0    0    -1
+$EndComp
+$Comp
+L LED:WS2812B D50
+U 1 1 5FA26D5C
+P 6450 4900
+F 0 "D50" H 6794 4946 50  0000 L CNN
+F 1 "WS2812B" H 6794 4855 50  0000 L CNN
+F 2 "LED_SMD:LED_WS2812B_PLCC4_5.0x5.0mm_P3.2mm" H 6500 4600 50  0001 L TNN
+F 3 "https://cdn-shop.adafruit.com/datasheets/WS2812B.pdf" H 6550 4525 50  0001 L TNN
+	1    6450 4900
+	1    0    0    -1
+$EndComp
+$Comp
+L LED:WS2812B D49
+U 1 1 5FA335D0
+P 5500 4900
+F 0 "D49" H 5844 4946 50  0000 L CNN
+F 1 "WS2812B" H 5844 4855 50  0000 L CNN
+F 2 "LED_SMD:LED_WS2812B_PLCC4_5.0x5.0mm_P3.2mm" H 5550 4600 50  0001 L TNN
+F 3 "https://cdn-shop.adafruit.com/datasheets/WS2812B.pdf" H 5600 4525 50  0001 L TNN
+	1    5500 4900
+	1    0    0    -1
+$EndComp
+Wire Wire Line
+	7100 4900 6750 4900
+Wire Wire Line
+	6150 4900 5800 4900
+$Comp
+L power:GND #PWR0114
+U 1 1 5FA579A8
+P 5500 5200
+F 0 "#PWR0114" H 5500 4950 50  0001 C CNN
+F 1 "GND" H 5505 5027 50  0000 C CNN
+F 2 "" H 5500 5200 50  0001 C CNN
+F 3 "" H 5500 5200 50  0001 C CNN
+	1    5500 5200
+	1    0    0    -1
+$EndComp
+$Comp
+L power:GND #PWR0115
+U 1 1 5FA58F2F
+P 6450 5200
+F 0 "#PWR0115" H 6450 4950 50  0001 C CNN
+F 1 "GND" H 6455 5027 50  0000 C CNN
+F 2 "" H 6450 5200 50  0001 C CNN
+F 3 "" H 6450 5200 50  0001 C CNN
+	1    6450 5200
+	1    0    0    -1
+$EndComp
+$Comp
+L power:GND #PWR0116
+U 1 1 5FA5976D
+P 7400 5200
+F 0 "#PWR0116" H 7400 4950 50  0001 C CNN
+F 1 "GND" H 7405 5027 50  0000 C CNN
+F 2 "" H 7400 5200 50  0001 C CNN
+F 3 "" H 7400 5200 50  0001 C CNN
+	1    7400 5200
+	1    0    0    -1
+$EndComp
+$Comp
+L power:+5V #PWR0117
+U 1 1 5FA5A4AF
+P 7400 4600
+F 0 "#PWR0117" H 7400 4450 50  0001 C CNN
+F 1 "+5V" H 7415 4773 50  0000 C CNN
+F 2 "" H 7400 4600 50  0001 C CNN
+F 3 "" H 7400 4600 50  0001 C CNN
+	1    7400 4600
+	1    0    0    -1
+$EndComp
 $EndSCHEMATC
